File: Hardware/status_leds/status_leds.kicad_pcb (KiCad board)
At the start: 2 copper layers, 18 parts, among them J1 Conn_01x18_Female, J2 Conn_01x04_Female, J3 Conn_01x08_Female

Commit message: hardware: update pcbs
Signed-off-by: Tillmann Heidsieck <theidsieck@leenox.de>
Parts:
- removed A1: Arduino_Nano_v2.x, Module:Arduino_Nano
- removed A2: DFPlayer, tonuino:DFPlayer
- removed J1: Conn_01x18_Female, Connector_PinHeader_2.54mm:PinHeader_1x18_P2.54mm_Vertical
- removed J3: Conn_01x08_Female, Connector_PinSocket_2.54mm:PinSocket_1x08_P2.54mm_Horizontal
- removed R1: 1k, Resistor_SMD:R_0402_1005Metric
- removed R2, R3, R4, R5: 4k7, Resistor_SMD:R_0402_1005Metric
- removed the REF** at (166.4, 81.3)
- removed the REF** at (193.0, 132.1)
- added REF**: OSHW-Logo2_7.3x6mm_SilkScreen, Symbol:OSHW-Logo2_7.3x6mm_SilkScreen, B.Cu at (191.8, 132.1)
Routing:
- net /3V3: track 56.5 -> 0.00 mm
- net /~HEADP: track 56.0 -> 0.00 mm
- net /~PAUSE: track 46.7 -> 0.00 mm, vias 1 -> 0
- net /~UP: track 42.8 -> 0.00 mm, vias 1 -> 0
- net /LED0: track 42.7 -> 0.00 mm
- net /RST: track 40.4 -> 0.00 mm
- net /LED1: track 40.1 -> 0.00 mm
- net /~DOWN: track 39.9 -> 0.00 mm, vias 1 -> 0
- net /SCK: track 39.6 -> 0.00 mm
- net /LED2: track 36.5 -> 0.00 mm
- net Net-(A1-Pad8): track 32.6 -> 0.00 mm
- net /MISO: track 29.4 -> 0.00 mm
- net /MOSI: track 27.0 -> 0.00 mm
- net /SS: track 23.0 -> 0.00 mm
- net Net-(A1-Pad5): track 18.7 -> 0.00 mm
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- removed copper zone on F.Cu, net /GND
- removed copper zone on B.Cu, net /VCC
Other:
- board outline added: 81.3 x 10.2 mm
- board text removed: "3V3"
- board text removed: "CS"
- board text removed: "D0"
- board text removed: "DWN"
- board text removed: "GND"
- board text removed: "HPL"
- board text removed: "HPP"
- board text removed: "HPR"
- board text removed: "MISO"
- board text removed: "MOSI"
- board text removed: "P/P"
- board text removed: "RST"
- board text removed: "SCK"
- board text removed: "SP+"
- board text removed: "SP-"
- board text removed: "UP"
- board text removed: "VIN"
